Commit message: Kalibrasyon hatti (calibrate.py, olcum sablonlari), simulasyon seçenekleri (robot_radius, sensor_noise_std, calibration), Pi 4 pin onerisi, URDF 133 mm, ROS testi ve yetim surec duzeltmesi
Co-Authored-By: Claude Sonnet 5.5 <noreply@anthropic.com>

File: src/arena_sim/urdf/pai_bot.urdf (robot description, URDF)
Before this commit: robot pai_bot, 9 links, 8 joints
Links:
- link base_link: geometry collision box size=0.133 0.09 0.04; visual box size=0.133 0.09 0.04
Joints:
- joint imu_joint: origin xyz=-0.02 0 0.02 rpy=0 0 0 -> xyz=-0.0185 0 0.02 rpy=0 0 0
