File: design/pcb/kicad/pico-carrier.kicad_sch (KiCad schematic)
At the start: 25 parts, among them J1 TB6612FNG modulu, sol sira, J10 S7V7F5 5 V regulator, J2 TB6612FNG modulu, sag sira, J3 TOF400C sol, J4 TOF400C orta, J5 TOF400C sag, J6 MPU6050 (GY-521), J7 Sol motor + enkoder, J8 Sag motor + enkoder, J9 Pil girisi 4xAA, SW1 Guc anahtari (harici), U1 Raspberry Pi Pico 2 W

Commit message: Tek katmanli Pico karti (55 x 58): konnektor siralari, tek tel kopru, Freerouting job_timeout, tek katman testleri
Co-Authored-By: Claude Sonnet 5.5 <noreply@anthropic.com>
Parts:
- removed C3: 10 uF, Capacitor_THT:CP_Radial_D5.0mm_P2.00mm, symbol pico-carrier:C3
- removed C5: 100 nF, Capacitor_THT:C_Disc_D5.0mm_W2.5mm_P5.00mm, symbol pico-carrier:C5
- removed J10: S7V7F5 5 V regulator, Connector_PinSocket_2.54mm:PinSocket_1x03_P2.54mm_Vertical, symbol pico-carrier:J10
- removed J2: TB6612FNG modulu, sag sira, Connector_PinSocket_2.54mm:PinSocket_1x08_P2.54mm_Vertical, symbol pico-carrier:J2
- removed J6: MPU6050 (GY-521), Connector_PinSocket_2.54mm:PinSocket_1x04_P2.54mm_Vertical, symbol pico-carrier:J6
- removed JP1: Sensor besleme secimi, Connector_PinHeader_2.54mm:PinHeader_1x03_P2.54mm_Vertical, symbol pico-carrier:JP1
- removed SW1: Guc anahtari (harici), Connector_PinHeader_2.54mm:PinHeader_1x02_P2.54mm_Vertical, symbol pico-carrier:SW1
- removed TP1: TP_3V3, Connector_PinHeader_2.54mm:PinHeader_1x01_P2.54mm_Vertical, symbol pico-carrier:TP1
- removed TP2: TP_5V, Connector_PinHeader_2.54mm:PinHeader_1x01_P2.54mm_Vertical, symbol pico-carrier:TP2
- removed TP3: TP_VM, Connector_PinHeader_2.54mm:PinHeader_1x01_P2.54mm_Vertical, symbol pico-carrier:TP3
- removed TP4: TP_GND, Connector_PinHeader_2.54mm:PinHeader_1x01_P2.54mm_Vertical, symbol pico-carrier:TP4
- added W2: Tel kopru 3V3, pico-carrier:WireLink_P30.48mm, symbol pico-carrier:W2
- C2: value 470 uF / 16 V -> 100 uF / 10 V; footprint Capacitor_THT:CP_Radial_D8.0mm_P3.50mm -> Capacitor_THT:CP_Radial_D6.3mm_P2.50mm
- D1: footprint Diode_THT:D_DO-41_SOD81_P10.16mm_Horizontal -> Diode_THT:D_DO-41_SOD81_P2.54mm_Vertical_KathodeUp
- J1: value TB6612FNG modulu, sol sira -> Surucu baglantisi (TB6612); footprint Connector_PinSocket_2.54mm:PinSocket_1x08_P2.54mm_Vertical -> Connector_PinHeader_2.54mm:PinHeader_1x10_P2.54mm_Vertical
- J7: value Sol motor + enkoder -> Sol enkoder; footprint Connector_PinHeader_2.54mm:PinHeader_1x06_P2.54mm_Vertical -> Connector_PinHeader_2.54mm:PinHeader_1x04_P2.54mm_Vertical
- J8: value Sag motor + enkoder -> Sag enkoder; footprint Connector_PinHeader_2.54mm:PinHeader_1x06_P2.54mm_Vertical -> Connector_PinHeader_2.54mm:PinHeader_1x04_P2.54mm_Vertical
- J9: value Pil girisi 4xAA -> LiPo girisi (1S); footprint TerminalBlock:TerminalBlock_bornier-2_P5.08mm -> Connector_JST:JST_PH_B2B-PH-K_1x02_P2.00mm_Vertical
- R1: value 20 k -> 100 k; footprint Resistor_THT:R_Axial_DIN0207_L6.3mm_D2.5mm_P10.16mm_Horizontal -> Resistor_THT:R_Axial_DIN0207_L6.3mm_D2.5mm_P2.54mm_Vertical
- R2: value 10 k -> 100 k; footprint Resistor_THT:R_Axial_DIN0207_L6.3mm_D2.5mm_P10.16mm_Horizontal -> Resistor_THT:R_Axial_DIN0207_L6.3mm_D2.5mm_P2.54mm_Vertical
Connections:
- net +5V is gone; now on net VBAT_SW: D1.2 (A)
- net VBAT_RAW is gone; now on net VBAT_SW: J9.1 (+)
- net +3V3: now also W2.1; no longer J1.2 (VCC), J7.3 (ENC_VCC), J8.3 (ENC_VCC)
- net AIN1: now also J1.2 (AIN1)
- net AIN2: now also J1.3 (AIN2)
- net BIN1: now also J1.4 (BIN1)
- net BIN2: now also J1.5 (BIN2)
- net ENC_L_A: now also J7.3 (ENC_A); no longer J7.5 (ENC_A)
- net ENC_L_B: now also J7.4 (ENC_B); no longer J7.6 (ENC_B)
- net ENC_R_A: now also J8.3 (ENC_A); no longer J8.5 (ENC_A)
- net ENC_R_B: now also J8.4 (ENC_B); no longer J8.6 (ENC_B)
- net GND: no longer C4.2, J1.3 (GND1), J3.2 (GND), J4.2 (GND), J5.2 (GND), J7.4 (ENC_GND), J8.4 (ENC_GND), U1.13 (GND_13), U1.18 (GND_18), U1.23 (GND_23), U1.28 (GND_28), U1.3 (GND_3), U1.33 (GND_33), U1.8 (GND_8)
- net PWMA: now also J1.1 (PWMA)
- net PWMB: now also J1.6 (PWMB)
- net STBY: now also J1.7 (STBY)
- net VBAT_SW: now also J1.10 (VM), J1.9 (VCC); no longer J1.1 (VM)
- net +SENS renamed GND_L
- net GND_L: now also C4.2, J7.1 (ENC_GND), J8.1 (ENC_GND), U1.3 (GND_3); no longer C4.1
- removed net MOT_L+: J1.4 (AO1), J7.1 (M+)
- net MOT_L- renamed +3V3_L
- net +3V3_L: now also C4.1, J3.2 (VIN), J4.2 (VIN), J5.2 (VIN), J8.2 (ENC_VCC), W2.2; no longer J1.5 (AO2)
- removed net MOT_R+: J1.7 (BO1), J8.1 (M+)
- removed net MOT_R-: J1.6 (BO2), J8.2 (M-)
- no-connect marks 13 -> 19
